File: HW/LED Controll Board/ctrl.kicad_pcb (KiCad board)
At the start: 2 copper layers, 0 parts

Commit message: W22812 Based design added
Parts:
- added C1: 470nF/10V, c_0805, F.Cu at (202.2, 147.1)
- added DP8049: , DP8049, F.Cu at (209.6, 152.4)
- added J0: LED00, CONN_NCW254-04S, F.Cu at (191.8, 170.2)
- added J1: LED01, CONN_NCW254-04S, F.Cu at (207.0, 170.2)
- added J10: LED10, CONN_NCW254-04S, F.Cu at (222.2, 134.6)
- added J11: LED11, CONN_NCW254-04S, F.Cu at (237.5, 134.6)
- added J12: LED12, CONN_NCW254-04S, F.Cu at (191.8, 134.6)
- added J13: LED13, CONN_NCW254-04S, F.Cu at (207.0, 134.6)
- added J14: LED14, CONN_NCW254-04S, F.Cu at (214.6, 134.6)
- added J15: LED15, CONN_NCW254-04S, F.Cu at (229.9, 134.6)
- added J16: PWR, CONN_NCW254-03S, F.Cu at (176.5, 141.0)
- added J17: SPI, HDR-6, F.Cu at (176.5, 156.2)
- added J2: LED02, CONN_NCW254-04S, F.Cu at (214.6, 170.2)
- added J3: LED03, CONN_NCW254-04S, F.Cu at (229.9, 170.2)
- added J4: LED04, CONN_NCW254-04S, F.Cu at (184.2, 170.2)
- added J5: LED05, CONN_NCW254-04S, F.Cu at (199.4, 170.2)
- added J6: LED06, CONN_NCW254-04S, F.Cu at (222.2, 170.2)
- added J7: LED07, CONN_NCW254-04S, F.Cu at (237.5, 170.2)
- added J8: LED08, CONN_NCW254-04S, F.Cu at (184.2, 134.6)
- added J9: LED09, CONN_NCW254-04S, F.Cu at (199.4, 134.6)
- added U1: TLC5955, HTSSOP-56, F.Cu at (210.8, 152.4)
Routing:
- net N-0000030: track 0.00 -> 166.3 mm
- net GND: track 0.00 -> 75.6 mm, vias 0 -> 11
- net N-0000031: track 0.00 -> 46.9 mm
- net N-0000033: track 0.00 -> 46.5 mm
- net N-0000026: track 0.00 -> 41.5 mm
- net N-0000044: track 0.00 -> 39.8 mm
- net N-0000035: track 0.00 -> 35.8 mm
- net N-0000014: track 0.00 -> 35.8 mm
- net N-0000025: track 0.00 -> 35.4 mm
- net N-0000027: track 0.00 -> 34.0 mm
- net N-0000045: track 0.00 -> 33.7 mm
- net N-0000055: track 0.00 -> 33.4 mm
- net N-000001: track 0.00 -> 33.1 mm
- net N-0000034: track 0.00 -> 32.9 mm
- net N-0000032: track 0.00 -> 32.6 mm, vias 0 -> 2
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- added copper zone on B.Cu, net GND
- added copper zone on F.Cu, net GND
Other:
- board outline added: 80 x 49 mm
- net class Default: clearance 0.254 -> 0.2
- rule trace_clearance: 0.254 -> 0.2
