File: HW/LED Controll Board/ctrl.sch (KiCad schematic (older format))
At the start: 0 parts

Commit message: W22812 Based design added
Parts:
- added C1: 470nF/10V, c_0805, symbol C
- added J0: LED00, CONN_NCW254-04S, symbol CONN_4
- added J1: LED01, CONN_NCW254-04S, symbol CONN_4
- added J10: LED10, CONN_NCW254-04S, symbol CONN_4
- added J11: LED11, CONN_NCW254-04S, symbol CONN_4
- added J12: LED12, CONN_NCW254-04S, symbol CONN_4
- added J13: LED13, CONN_NCW254-04S, symbol CONN_4
- added J14: LED14, CONN_NCW254-04S, symbol CONN_4
- added J15: LED15, CONN_NCW254-04S, symbol CONN_4
- added J16: PWR, CONN_NCW254-03S, symbol CONN_3
- added J17: SPI, HDR-6, symbol CONN_6
- added J2: LED02, CONN_NCW254-04S, symbol CONN_4
- added J3: LED03, CONN_NCW254-04S, symbol CONN_4
- added J4: LED04, CONN_NCW254-04S, symbol CONN_4
- added J5: LED05, CONN_NCW254-04S, symbol CONN_4
- added J6: LED06, CONN_NCW254-04S, symbol CONN_4
- added J7: LED07, CONN_NCW254-04S, symbol CONN_4
- added J8: LED08, CONN_NCW254-04S, symbol CONN_4
- added J9: LED09, CONN_NCW254-04S, symbol CONN_4
- added U1: TLC5955, HTSSOP-56, symbol TLC5955
Connections:
- net labels added: GND
- wire segments 0 -> 86
