File: HW/LED Stripe Neo/LED Stripe Neo.kicad_pcb (KiCad board)
At the start: 2 copper layers, 109 x 13.5 mm, 22 parts, among them J1 IN-OUT, J2 IN-OUT, U1 WS2812B, U10 WS2812B, U2 WS2812B, U3 WS2812B, U4 WS2812B, U5 WS2812B, U6 WS2812B, U7 WS2812B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

Commit message: Fix WS2812 vs WS2812B footprint differences
Parts:
- U1, U10, U2, U3, U4, U5, U6, U7, U8, U9: value WS2812B -> WS2812
